File: Underground-BMS.kicad_sch (KiCad schematic)
At the start: 132 parts, among them J1 EXT_ACT_BAL, J15 BQ_PROG, J2 BATT+, J25 SEL3V3, J26 12V+, J27 12V-, J29 VBATT, J3 BATT-, J4 Think-BMS-Connector, J5 EXT_PWR_BUS, J6 PROT_FET, J7 ISENSE, J8 XRES, J9 Imdrv, Q1 FCX495(Q)TA, Q2 BC847, U1 TMUX1309, U2 TMUX1309, U3 BQ7695204

Commit message: Restructuring and schematic floor plan
Parts:
- removed C1: 10u, Capacitor_SMD:C_0805_2012Metric_Pad1.18x1.45mm_HandSolder, symbol Device:C_Small
- removed C10, C11, C12, C13, C14, C15, C16, C17, C18, C19, C20, C22, C5, C6, C7, C8, C9: 220n, Capacitor_SMD:C_0603_1608Metric_Pad1.08x0.95mm_HandSolder, symbol Device:C_Small
- removed C2, C23, C25, C26, C27, C29, C33, C34, C35, C63, C64, C69: 100n, Capacitor_SMD:C_0603_1608Metric_Pad1.08x0.95mm_HandSolder, symbol Device:C_Small
- removed C21: 47u, Capacitor_SMD:C_0805_2012Metric_Pad1.18x1.45mm_HandSolder, symbol Device:C_Small
- removed C24, C4: 100p, Capacitor_SMD:C_0603_1608Metric_Pad1.08x0.95mm_HandSolder, symbol Device:C_Small
- removed C28, C30, C32: 2u2, Capacitor_SMD:C_0805_2012Metric_Pad1.18x1.45mm_HandSolder, symbol Device:C_Small
- removed C3: 1u, Capacitor_SMD:C_0805_2012Metric_Pad1.18x1.45mm_HandSolder, symbol Device:C_Small
- removed C31: 22n, Capacitor_SMD:C_0603_1608Metric_Pad1.08x0.95mm_HandSolder, symbol Device:C_Small
- removed D1, D2: SS 16, Diode_SMD:D_SMA-SMB_Universal_Handsoldering, symbol Device:D_Schottky
- removed D3: ALERT, LED_SMD:LED_0603_1608Metric_Pad1.05x0.95mm_HandSolder, symbol Device:LED_Small
- removed H1, H2, H3, H4: MountingHole, MountingHole:MountingHole_5.5mm, symbol Mechanical:MountingHole
- removed J1: EXT_ACT_BAL, Connector_IDC:IDC-Header_2x20_P2.54mm_Vertical, symbol Connector_Generic:Conn_02x20_Odd_Even
- removed J15: BQ_PROG, Connector_PinHeader_2.54mm:PinHeader_1x05_P2.54mm_Vertical, symbol Connector_Generic:Conn_01x05
- removed J2: BATT+, the78mole:WE-WP-PLUG_REDCUBE, symbol Connector_Generic:Conn_01x01
- removed J25: SEL3V3, Connector_PinHeader_2.54mm:PinHeader_1x03_P2.54mm_Vertical, symbol Connector_Generic:Conn_01x03
- removed J26: 12V+, the78mole:WE-WP-PLUG_REDCUBE, symbol Connector_Generic:Conn_01x01
- removed J27: 12V-, the78mole:WE-WP-PLUG_REDCUBE, symbol Connector_Generic:Conn_01x01
- removed J29: VBATT, Connector_JST:JST_XH_S2B-XH-A_1x02_P2.50mm_Horizontal, symbol Connector_Generic:Conn_01x02
- removed J3: BATT-, the78mole:WE-WP-PLUG_REDCUBE, symbol Connector_Generic:Conn_01x01
- removed J4: Think-BMS-Connector, the78mole:Think-BMS-Connector, symbol the78mole:Think-BMS-Connector
- removed J5: EXT_PWR_BUS, Connector_IDC:IDC-Header_2x10_P2.54mm_Vertical, symbol Connector_Generic:Conn_02x10_Odd_Even
- removed J6: PROT_FET, Connector_IDC:IDC-Header_2x05_P2.54mm_Vertical, symbol Connector_Generic:Conn_01x10
- removed J7: ISENSE, Connector_JST:JST_PH_B4B-PH-K_1x04_P2.00mm_Vertical, symbol Connector_Generic:Conn_01x04
- removed J8: XRES, Connector_JST:JST_PH_B2B-PH-K_1x02_P2.00mm_Vertical, symbol Connector_Generic:Conn_01x02
- removed J9: Imdrv, Connector_PinHeader_2.54mm:PinHeader_1x03_P2.54mm_Vertical, symbol Connector_Generic:Conn_01x03
- removed Q1: FCX495(Q)TA, Package_TO_SOT_SMD:SOT-89-3_Handsoldering, symbol Device:Q_NPN_BCE
- removed Q2: BC847, Package_TO_SOT_SMD:SOT-23, symbol Transistor_BJT:BC847
- removed R1, R2, R3: 47K, Resistor_SMD:R_0603_1608Metric_Pad0.98x0.95mm_HandSolder, symbol Device:R_Small
- removed R10, R11, R12, R13, R14, R15, R16, R17, R18, R19, R20, R21, R22, R6, R7, R8, R9: 22, Resistor_SMD:R_0603_1608Metric_Pad0.98x0.95mm_HandSolder, symbol Device:R_Small
- removed R100, R24, R29, R30, R31, R32, R4, R46, R47, R5, R93, R94, R95, R96, R97, R98, R99: NP, Resistor_SMD:R_0603_1608Metric_Pad0.98x0.95mm_HandSolder, symbol Device:R_Small
- removed R106, R107, R50, R51, R52, R53, R54, R55, R56, R57, R58: 33, Resistor_SMD:R_0603_1608Metric_Pad0.98x0.95mm_HandSolder, symbol Device:R_Small
- removed R23, R27, R28: 100, Resistor_SMD:R_0603_1608Metric_Pad0.98x0.95mm_HandSolder, symbol Device:R_Small
- removed R25, R26, R45, R48: 10K, Resistor_SMD:R_0603_1608Metric_Pad0.98x0.95mm_HandSolder, symbol Device:R_Small
- removed R33, R34, R35, R36: 0, Resistor_SMD:R_0603_1608Metric_Pad0.98x0.95mm_HandSolder, symbol Device:R_Small
- removed R37, R38, R39, R40, R41, R42, R43, R44: 3K3, Resistor_SMD:R_0603_1608Metric_Pad0.98x0.95mm_HandSolder, symbol Device:R_Small
- removed R49: 1K, Resistor_SMD:R_0603_1608Metric_Pad0.98x0.95mm_HandSolder, symbol Device:R_Small
- removed U1, U2: TMUX1309, Package_SO:TSSOP-16_4.4x5mm_P0.65mm, symbol the78mole:TMUX1309
- removed U3: BQ7695204, Package_QFP:TQFP-48_7x7mm_P0.5mm, symbol the78mole:BQ7695204
Connections:
- no-connect marks 7 -> 0
Other:
- added sheet Active-Balancer (Active-Balancer.kicad_sch)
- added sheet BMS-Main (BMS-Main.kicad_sch)
- added sheet Current-Sense (Current-Sense.kicad_sch)
- added sheet ESP-Prog (ESP-Prog.kicad_sch)
- added sheet Protection (Protection.kicad_sch)
- added sheet RS485-Interface (RS485-Interface.kicad_sch)
- sheet CAN-Interface ports: added none; removed 3V3Logic, Board12V, BoardGND, CAN_RX, CAN_TX, CAN_nEN
- sheet ESP-Control ports: added none; removed 3V3_ESP, CAN_RX, CAN_TX, CAN_nEN, ESP_ADC1_CH0, ESP_ADC1_CH3, ESP_ADC1_CH4, ESP_ADC1_CH5, ESP_ALARM, ESP_AMUX_A0, ESP_AMUX_A1, ESP_AMUX_nEN, ESP_GPIO23, ESP_GPIO25, ESP_GPIO26, ESP_MISO, ESP_MOSI, ESP_SCL, ESP_SCLK, ESP_SDA, ESP_SHUT, ESP_nCS, ESP_nINT, ESP_nRESET
- sheet Power-Supply ports: added none; removed 3V3_OUT, PGOOD, PRE_5V_OUT, VIN
- note removed: "(1)"
- note removed: "1) It's not advised to use R4/R5 to supply the board. Better get battery power through seperate connectors/wires (J2/J3 or J4-A7/A8/B6/B7)."
- note removed: "Links: - https://randomnerdtutorials.com/esp32-i2c-communication-arduino-ide/"
- note removed: "Resistor swap for use of ISO1042 (swapped RX/TX comapred to ISO1050)"
- note removed: "The TMUX is hardly available in standard packages (TSSOP) and all other package options are non-standard, so we added a non-muxed fallback option."
